Commit message: added 3x revolute joints for each shoulder, and the .stl's for hands

File: pair_of_arms.urdf (robot description, URDF)
Before this commit: robot pair_of_arms, 7 links, 6 joints
Links:
- added link left_shoulder_pitch_link, mass 0.001; collision sphere radius=0.01; visual sphere radius=0.01
- added link left_shoulder_roll_link, mass 0.001; collision sphere radius=0.01; visual sphere radius=0.01
- added link right_shoulder_pitch_link, mass 0.001; collision sphere radius=0.01; visual sphere radius=0.01
- added link right_shoulder_roll_link, mass 0.001; collision sphere radius=0.01; visual sphere radius=0.01
Joints:
- removed joint left_shoulder_joint
- removed joint right_shoulder_joint
- added joint left_shoulder_pitch: type revolute, parent left_shoulder_pitch_link, child left_shoulder_roll_link, origin xyz=0 0 0 rpy=0 0 0, axis 0 1 0, limit lower=-1.57 upper=1.57 effort=100.0 velocity=0.5
- added joint left_shoulder_roll: type revolute, parent left_shoulder_roll_link, child left_upper_arm, origin xyz=0 0 0 rpy=0 0 0, axis 1 0 0, limit lower=-3.14 upper=3.14 effort=100.0 velocity=0.5
- added joint left_shoulder_yaw: type revolute, parent base_link, child left_shoulder_pitch_link, origin xyz=-0.25 0 0 rpy=0.8 0 0, axis 0 0 1, limit lower=-3.14 upper=3.14 effort=100.0 velocity=0.5
- added joint right_shoulder_pitch: type revolute, parent right_shoulder_pitch_link, child right_shoulder_roll_link, origin xyz=0 0 0 rpy=0 0 0, axis 0 1 0, limit lower=-1.57 upper=1.57 effort=100.0 velocity=0.5
- added joint right_shoulder_roll: type revolute, parent right_shoulder_roll_link, child right_upper_arm, origin xyz=0 0 0 rpy=0 0 0, axis 1 0 0, limit lower=-3.14 upper=3.14 effort=100.0 velocity=0.5
- added joint right_shoulder_yaw: type revolute, parent base_link, child right_shoulder_pitch_link, origin xyz=0.25 0 0 rpy=0.8 0 0, axis 0 0 1, limit lower=-3.14 upper=3.14 effort=100.0 velocity=0.5
